File: Hardware/KiCad/NudgePCB/NudgeEMGStrip/NudgeFlexStrip.kicad_pcb (KiCad board)
At the start: 2 copper layers, 48.5 x 174 mm, 18 parts, among them J1 Conn_01x17, J3 Conn_01x12, U1 ADS1298xPAG

Commit message: EMG strip: put VCAP3's 1uF capacitor directly on the pin (C7 -> 0 ohm R2)
The ADS1298 datasheet asks for 1uF from VCAP3 to AVSS; C7 (0.1uF) in series
with C3 (1uF) gave about 0.09uF. Same 0603 footprint position, so this is a
BOM change only. DRC and schematic parity unchanged.

Co-Authored-By: Claude Opus 5.5 (1M context) <noreply@anthropic.com>
Parts:
- R2: renamed from C7; value .1uF -> 0; footprint Capacitor_SMD:C_0603_1608Metric -> Resistor_SMD:R_0603_1608Metric
Changed lines of the file:
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@@
 		)
 	)
-	(footprint "Capacitor_SMD:C_0603_1608Metric"
+	(footprint "Resistor_SMD:R_0603_1608Metric"
 		(layer "F.Cu")
 		(at 75.775 87.5)
-		(descr "Capacitor SMD 0603 (1608 Metric), square (rectangular) end terminal, IPC-7351 nominal, (Body size source: IPC-SM-782 page 76, https://www.pcb-3d.com/wordpress/wp-content/uploads/ipc-sm-782a_amendment_1_and_2.pdf)")
-		(tags "capacitor")
-		(property "Reference" "C7"
+		(descr "Resistor SMD 0603 (1608 Metric), square (rectangular) end terminal, IPC-7351 nominal, (Body size source: IPC-SM-782 page 72, https://www.pcb-3d.com/wordpress/wp-content/uploads/ipc-sm-782a_amendment_1_and_2.pdf)")
+		(tags "resistor")
+		(property "Reference" "R2"
 			(at 0 -1.43 0)
 			(layer "F.SilkS")
@@
 			)
 		)
-		(property "Value" ".1uF"
+		(property "Value" "0"
 			(at 0 1.43 0)
 			(layer "F.Fab")
@@
 			)
 		)
-		(property "Description" "Unpolarized capacitor"
+		(property "Description" "0 ohm jumper: puts C3 (1uF) directly on VCAP3 as the ADS1298 datasheet requires (was 0.1uF in series)"
 			(at 0 0 0)
 			(layer "F.Fab")
@@
 			)
 		)
-		(property ki_fp_filters "C_*")
+		(property ki_fp_filters "R_*")
 		(sheetname "/")
 		(sheetfile "NudgeFlexStrip.kicad_sch")
@@
 		(duplicate_pad_numbers_are_jumpers no)
 		(fp_line
-			(start -0.14058 -0.51)
-			(end 0.14058 -0.51)
+			(start -0.237258 -0.5225)
+			(end 0.237258 -0.5225)
 			(stroke
 				(width 0.12)
@@
 		)
 		(fp_line
-			(start -0.14058 0.51)
-			(end 0.14058 0.51)
+			(start -0.237258 0.5225)
+			(end 0.237258 0.5225)
 			(stroke
 				(width 0.12)
@@
 		)
 		(fp_rect
-			(start -0.8 -0.4)
-			(end 0.8 0.4)
+			(start -0.8 -0.4125)
+			(end 0.8 0.4125)
 			(stroke
 				(width 0.1)
@@
 		)
 		(pad "1" smd roundrect
-			(at -0.775 0)
-			(size 0.9 0.95)
+			(at -0.825 0)
+			(size 0.8 0.95)
 			(layers "F.Cu" "F.Mask" "F.Paste")
 			(roundrect_rratio 0.25)
@@
 		)
 		(pad "2" smd roundrect
-			(at 0.775 0)
-			(size 0.9 0.95)
+			(at 0.825 0)
+			(size 0.8 0.95)
 			(layers "F.Cu" "F.Mask" "F.Paste")
 			(roundrect_rratio 0.25)
@@
 		)
 		(embedded_fonts no)
-		(model "${KICAD10_3DMODEL_DIR}/Capacitor_SMD.3dshapes/C_0603_1608Metric.step"
+		(model "${KICAD10_3DMODEL_DIR}/Resistor_SMD.3dshapes/R_0603_1608Metric.step"
 			(offset
 				(xyz 0 0 0)
