File: Hardware/KiCad/NudgePCB/NudgeEMGStrip/NudgeFlexStrip.kicad_sch (KiCad schematic)
At the start: 18 parts, among them J1 Conn_01x17, J3 Conn_01x12, U1 ADS1298xPAG

Commit message: EMG strip: put VCAP3's 1uF capacitor directly on the pin (C7 -> 0 ohm R2)
The ADS1298 datasheet asks for 1uF from VCAP3 to AVSS; C7 (0.1uF) in series
with C3 (1uF) gave about 0.09uF. Same 0603 footprint position, so this is a
BOM change only. DRC and schematic parity unchanged.

Co-Authored-By: Claude Opus 5.5 (1M context) <noreply@anthropic.com>
Parts:
- removed C7: .1uF, Capacitor_SMD:C_0603_1608Metric, symbol Device:C
- added R2: 0, Resistor_SMD:R_0603_1608Metric, symbol Device:R
Connections:
- net at C3.2: now also R2.1
- net at U1.55 (VCAP3): now also R2.2
Changed lines of the file:
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@@
-	)
-	(symbol
-		(lib_id "Device:C")
-		(at 40.64 146.05 90)
-		(unit 1)
-		(body_style 1)
-		(exclude_from_sim no)
-		(in_bom yes)
-		(on_board yes)
-		(in_pos_files yes)
-		(dnp no)
-		(property "Reference" "C7"
-			(at 40.64 138.43 90)
-			(show_name no)
-			(do_not_autoplace no)
-			(effects
-				(font
-					(size 1.27 1.27)
-				)
-			)
-		)
-		(property "Value" ".1uF"
-			(at 40.386 148.844 90)
-			(show_name no)
-			(do_not_autoplace no)
-			(effects
-				(font
-					(size 1.27 1.27)
-				)
-			)
-		)
-		(property "Footprint" "Capacitor_SMD:C_0603_1608Metric"
-			(at 44.45 145.0848 0)
-			(hide yes)
-			(show_name no)
-			(do_not_autoplace no)
-			(effects
-				(font
-					(size 1.27 1.27)
-				)
-			)
-		)
-		(property "Datasheet" ""
-			(at 40.64 146.05 0)
-			(hide yes)
-			(show_name no)
-			(do_not_autoplace no)
-			(effects
-				(font
-					(size 1.27 1.27)
-				)
-			)
-		)
-		(property "Description" "Unpolarized capacitor"
-			(at 40.64 146.05 0)
-			(hide yes)
-			(show_name no)
-			(do_not_autoplace no)
-			(effects
-				(font
-					(size 1.27 1.27)
-				)
-			)
-		)
-		(pin "2"
-		)
-		(pin "1"
-		)
-		(instances
-			(project "NudgeFlexStrip"
-				(path "/4e1ae81a-3816-4b95-8645-dc2f32948656"
-					(reference "C7")
-					(unit 1)
-				)
-			)
-		)
 	)
 	(symbol
@@
 		)
 	)
-	(sheet_instances
+	  (symbol (lib_id "Device:R") (at 40.64 146.05 90) (unit 1)
+    (body_style 1) (exclude_from_sim no) (in_bom yes) (on_board yes) (in_pos_files yes) (dnp no)
+    (property "Reference" "R2"
+      (at 40.64 144.018 90)
+      (show_name no)
+      (do_not_autoplace no)
+      (effects
+					(font
+						(size 1.27 1.27)
+					)
+				)
+    )
+    (property "Value" "0"
+      (at 40.64 146.05 90)
+      (show_name no)
+      (do_not_autoplace no)
+      (effects
+					(font
+						(size 1.27 1.27)
+					)
+				)
+    )
+    (property "Footprint" "Resistor_SMD:R_0603_1608Metric"
+      (at 40.64 147.828 90)
+      (hide yes)
+      (show_name no)
+      (do_not_autoplace no)
+      (effects
+					(font
+						(size 1.27 1.27)
+					)
+				)
+    )
+    (property "Datasheet" ""
+      (at 40.64 146.05 0)
+      (hide yes)
+      (show_name no)
+      (do_not_autoplace no)
+      (effects
+					(font
+						(size 1.27 1.27)
+					)
+				)
+    )
+    (property "Description" "0 ohm jumper: puts C3 (1uF) directly on VCAP3 as the ADS1298 datasheet requires (was 0.1uF in series)"
+      (at 40.64 146.05 0)
+      (hide yes)
+      (show_name no)
+      (do_not_autoplace no)
+      (effects
+					(font
+						(size 1.27 1.27)
+					)
+				)
+    )
+    (pin "1")
+    (pin "2")
+    (instances
+      (project "NudgeFlexStrip"
+        (path "/4e1ae81a-3816-4b95-8645-dc2f32948656"
+          (reference "R2")
+          (unit 1)
+        )
+      )
+    )
+  )
+  (sheet_instances
 		(path "/"
 			(page "1")
