File: Hardware/KiCad/NudgePCB/Nudge/Nudge.kicad_sch (KiCad schematic)
At the start: 29 parts, among them J1 Conn_01x02, J2 Conn_01x03, J3 Conn_01x02, J4 Conn_01x02, J5 Conn_01x06, J6 Conn_01x06, SW1 SW_SPST, U1 XIAO-ESP32-S3-SMD

Commit message: Main board schematic: EMG strip connector replaces the MyoWare connector
J2 becomes a 12-pin header wired 1:1 to the strip's J3 (ADS1298): SPI on the
XIAO ESP32-S3 bottom pads (MTCK=SCLK, MTDO=DIN, MTDI=DOUT, MTMS=CS), DRDY on
D0, CLKSEL/PWDN/RESET tied to 3V3, START to GND. Matches BoardConfig.h.
Also points the glove symbol library at the copy in the repo instead of a
path on another machine. ERC: 0 violations. PCB not updated yet.

Co-Authored-By: Claude Opus 5.5 (1M context) <noreply@anthropic.com>
Parts:
- removed J2: Conn_01x03, Connector_JST:JST_PH_S3B-PH-K_1x03_P2.00mm_Horizontal, symbol Connector_Generic:Conn_01x03
- added J2: EMG_Strip, Connector_PinHeader_2.54mm:PinHeader_1x12_P2.54mm_Vertical, symbol Connector_Generic:Conn_01x12
Connections:
- net +3V3: now also J2.1 (Pin_1), J2.10 (Pin_10), J2.11 (Pin_11), J2.7 (Pin_7)
- net GND: now also J2.12 (Pin_12), J2.8 (Pin_8)
- net STRIP_DOUT: now reaches U1.15 (MTDI)
- net STRIP_DOUT: now also J2.5 (Pin_5)
- net STRIP_DIN: now reaches U1.16 (MTDO)
- net STRIP_DIN: now also J2.3 (Pin_3)
- net STRIP_CS: now reaches U1.19 (MTMS)
- net STRIP_CS: now also J2.4 (Pin_4)
- net STRIP_SCLK: now reaches U1.20 (MTCK)
- net STRIP_SCLK: now also J2.2 (Pin_2)
- net EMG renamed STRIP_DRDY
- net STRIP_DRDY: now also J2.9 (Pin_9)
- no-connect marks 18 -> 15
Other:
- note added: "8. EMG strip (replaces MyoWare J2) 1:1 cable to the strip's J3 (ADS1298). CLKSEL, PWDN, RESET tied high; START low; CLK unused. SPI on the XIAO bottom pads."
